File: 40pin_AVRMCU.sch (KiCad schematic (older format))
At the start: 21 parts, among them IC1 ATMEGA32-A, P1 CONN_5X2, P2 CONN_10, P3 CONN_10, P4 CONN_10, P5 CONN_10, P6 CONN_7, P7 CONN_01X01, SW1 rst, X1 16Mhz

Commit message: Updated designs
Parts:
- removed C1: 0.1uF, symbol C
- removed P6: CONN_7, symbol CONN_7
- added C7, C8, C9: 0.1uF, symbol C
- added CON1: USB-MINI-B, symbol USB-MINI-B
- added P10, P6, P8, P9: CONN_01X01, symbol CONN_01X01
- added R4, R5: R, symbol R
- added U1: CP2102, symbol CP2102
Connections:
- net +5V: now also C7.2, CON1.1 (VBUS), U1.7 (REGIN), U1.8 (VBUS); no longer C4.1, IC1.29 (AREF)
- net GND: now also C7.1, C8.2
- net RX: now also R5.1
- net TX: now also R4.1
- net rst: now also C9.1
- net Aref: now reaches P2.1 (P1)
- net Aref: now also C4.1, IC1.29 (AREF)
- net SCL: now reaches IC1.19 ((SCL)PC0), P4.1 (P1)
- net SCL: now also P4.10 (P10)
- net SDA: now reaches IC1.20 ((SDA)PC1), P4.2 (P2)
- net SDA: now also P4.9 (P9)
- new net: CON1.2 (D-), U1.5 (D-)
- new net: CON1.3 (D+), U1.4 (D+)
- new net: CON1.4 (ID), U1.3 (GND)
- new net: R4.2, U1.25 (RXD)
- new net: R5.2, U1.26 (TXD)
- new net: C9.2, U1.28 (DTR)
- new net: C8.1, U1.6 (VDD)
- no-connect marks 7 -> 29
Other:
- moved on the sheet: C2, C3, C4, C5, C6, D1, D3, IC1, P1, P2, P3, P4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

Commit message: updated
Parts:
- R4, R5: value R -> 470
Connections:
- net GND: now also CON1.5 (GND), U1.3 (GND)
- net at CON1.4 (ID): no longer U1.3 (GND)
Other:
- note added: "Logo"
- note added: "Mounting Holes"
Changed lines of the file:
@@
 NoConn ~ 8225 1275
 $Comp
-L GND #PWR10
+L GND #PWR01
 U 1 1 54F1C118
 P 9025 1625
-F 0 "#PWR10" H 9025 1625 30  0001 C CNN
+F 0 "#PWR01" H 9025 1625 30  0001 C CNN
 F 1 "GND" H 9025 1555 30  0001 C CNN
 F 2 "" H 9025 1625 60  0001 C CNN
@@
 $EndComp
 $Comp
-L GND #PWR6
+L GND #PWR02
 U 1 1 54F1C142
 P 3025 3150
-F 0 "#PWR6" H 3025 3150 30  0001 C CNN
+F 0 "#PWR02" H 3025 3150 30  0001 C CNN
 F 1 "GND" H 3025 3080 30  0001 C CNN
 F 2 "" H 3025 3150 60  0001 C CNN
@@
 $EndComp
 $Comp
-L GND #PWR8
+L GND #PWR03
 U 1 1 54F1C14E
 P 4725 1050
-F 0 "#PWR8" H 4725 1050 30  0001 C CNN
+F 0 "#PWR03" H 4725 1050 30  0001 C CNN
 F 1 "GND" H 4725 980 30  0001 C CNN
 F 2 "" H 4725 1050 60  0001 C CNN
@@
 rst
 $Comp
-L GND #PWR7
+L GND #PWR04
 U 1 1 54F1C15B
 P 4175 5250
-F 0 "#PWR7" H 4175 5250 30  0001 C CNN
+F 0 "#PWR04" H 4175 5250 30  0001 C CNN
 F 1 "GND" H 4175 5180 30  0001 C CNN
 F 2 "" H 4175 5250 60  0001 C CNN
@@
 $EndComp
 $Comp
-L GND #PWR3
+L GND #PWR05
 U 1 1 54F1C161
 P 2325 2050
-F 0 "#PWR3" H 2325 2050 30  0001 C CNN
+F 0 "#PWR05" H 2325 2050 30  0001 C CNN
 F 1 "GND" H 2325 1980 30  0001 C CNN
 F 2 "" H 2325 2050 60  0001 C CNN
@@
 $EndComp
 $Comp
-L GND #PWR2
+L GND #PWR06
 U 1 1 54F1C1A9
 P 1675 4375
-F 0 "#PWR2" H 1675 4375 30  0001 C CNN
+F 0 "#PWR06" H 1675 4375 30  0001 C CNN
 F 1 "GND" H 1675 4305 30  0001 C CNN
 F 2 "" H 1675 4375 60  0001 C CNN
@@
 	5675 1250 6225 1250
 $Comp
-L GND #PWR9
+L GND #PWR07
 U 1 1 54F1DF71
 P 5975 1200
-F 0 "#PWR9" H 5975 1200 30  0001 C CNN
+F 0 "#PWR07" H 5975 1200 30  0001 C CNN
 F 1 "GND" H 5975 1130 30  0001 C CNN
 F 2 "" H 5975 1200 60  0001 C CNN
@@
 	1675 1325 1675 1425
 $Comp
-L GND #PWR1
+L GND #PWR08
 U 1 1 54F94C89
 P 1675 1925
-F 0 "#PWR1" H 1675 1925 30  0001 C CNN
+F 0 "#PWR08" H 1675 1925 30  0001 C CNN
 F 1 "GND" H 1675 1855 30  0001 C CNN
 F 2 "" H 1675 1925 60  0001 C CNN
@@
 	8475 2300 8575 2300
 $Comp
-L GND #PWR11
+L GND #PWR09
 U 1 1 5514EEA3
 P 9175 2350
-F 0 "#PWR11" H 9175 2350 30  0001 C CNN
+F 0 "#PWR09" H 9175 2350 30  0001 C CNN
 F 1 "GND" H 9175 2280 30  0001 C CNN
 F 2 "" H 9175 2350 60  0001 C CNN
@@
 Text Notes 8450 2075 0    60   ~ 0
 TX LED
-Text Notes 8025 3175 0    60   ~ 0
+Text Notes 2500 5350 0    60   ~ 0
 Breakout for USB to Serial
 Text Notes 1375 650  0    60   ~ 0
@@
 Wire Wire Line
 	2350 6550 2950 6550
-Wire Wire Line
-	2350 6650 2950 6650
 $Comp
 L C C8
@@
 	3400 7300 3250 7300
 $Comp
-L GND #PWR5
+L GND #PWR010
 U 1 1 579B2EBF
 P 2700 7350
-F 0 "#PWR5" H 2700 7350 30  0001 C CNN
+F 0 "#PWR010" H 2700 7350 30  0001 C CNN
 F 1 "GND" H 2700 7280 30  0001 C CNN
 F 2 "" H 2700 7350 60  0001 C CNN
@@
 Connection ~ 2950 5500
 $Comp
-L GND #PWR4
+L GND #PWR011
 U 1 1 579B3413
 P 2650 6050
-F 0 "#PWR4" H 2650 6050 30  0001 C CNN
+F 0 "#PWR011" H 2650 6050 30  0001 C CNN
 F 1 "GND" H 2650 5980 30  0001 C CNN
 F 2 "" H 2650 6050 60  0001 C CNN
@@
 NoConn ~ 5300 6650
 NoConn ~ 3500 7300
-NoConn ~ 2350 6750
 NoConn ~ 1350 6350
 NoConn ~ 1350 6450
@@
 $EndComp
 $Comp
-L R R4
-U 1 1 579B39E3
-P 5600 6350
-F 0 "R4" V 5680 6350 50  0000 C CNN
-F 1 "R" V 5607 6351 50  0000 C CNN
-F 2 "" V 5530 6350 30  0000 C CNN
-F 3 "" H 5600 6350 30  0000 C CNN
-	1    5600 6350
-	0    1    1    0
-$EndComp
-$Comp
 L R R5
 U 1 1 579B3A3A
 P 5950 6450
 F 0 "R5" V 6030 6450 50  0000 C CNN
-F 1 "R" V 5957 6451 50  0000 C CNN
+F 1 "470" V 5957 6451 50  0000 C CNN
 F 2 "" V 5880 6450 30  0000 C CNN
 F 3 "" H 5950 6450 30  0000 C CNN
@@
 $EndComp
 Wire Wire Line
-	5300 6350 5350 6350
-Wire Wire Line
 	5300 6450 5700 6450
-Text Label 5850 6350 0    60   ~ 0
+Text Label 5950 6350 0    60   ~ 0
 TX
 Text Label 6200 6450 0    60   ~ 0
@@
 NoConn ~ 9725 5100
 NoConn ~ 10400 5100
+$Comp
+L GND #PWR012
+U 1 1 579C3353
+P 2350 6750
+F 0 "#PWR012" H 2350 6750 30  0001 C CNN
+F 1 "GND" H 2350 6680 30  0001 C CNN
+F 2 "" H 2350 6750 60  0001 C CNN
+F 3 "" H 2350 6750 60  0001 C CNN
+	1    2350 6750
+	1    0    0    -1
+$EndComp
+Wire Wire Line
+	2350 6750 2950 6750
+Wire Wire Line
+	2950 6750 2950 6650
+Text Notes 9000 4150 0    60   ~ 0
+Logo
+Text Notes 10000 4100 0    60   ~ 0
+Mounting Holes
+NoConn ~ 2350 6650
+$Comp
+L R R4
+U 1 1 579C4A4D
+P 5700 6350
+F 0 "R4" V 5780 6350 50  0000 C CNN
+F 1 "470" V 5707 6351 50  0000 C CNN
+F 2 "" V 5630 6350 30  0000 C CNN
+F 3 "" H 5700 6350 30  0000 C CNN
+	1    5700 6350
+	0    1    1    0
+$EndComp
+Wire Wire Line
+	5300 6350 5450 6350
 $EndSCHEMATC
