File: DesignFiles/40pin_AVRMCU.kicad_pcb (KiCad board)
At the start: 2 copper layers, 25.4 x 62.9 mm, 30 parts, among them CON1 USB-MINI-B, IC1 ATMEGA32-A, P1 CONN_5X2, P10 CONN_01X01, P2 CONN_10, P3 CONN_10, P4 CONN_10, P5 CONN_10, P6 CONN_01X01, P7 CONN_01X01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

Commit message: Changes done
Parts:
- CON1: footprint EE:USB_Micro-B_SMD_NEW -> Explore:USB_Micro-B_SMD_NEW_1
- D1, D3: footprint EE:LED-0603_NEW -> Explore:LED-0603_NEW
- IC1: footprint Housings_QFP:LQFP-44_10x10mm_Pitch0.8mm -> Housings_QFP:TQFP-44_10x10mm_Pitch0.8mm
- P1: footprint Pin_Headers:Pin_Header_Straight_2x05 -> Pin_Headers:Pin_Header_Straight_2x05_Pitch2.54mm
- P2, P3, P4, P5: footprint Pin_Headers:Pin_Header_Straight_1x10 -> Pin_Headers:Pin_Header_Straight_1x10_Pitch2.54mm
- P7: footprint Logo_new:Logo_8 -> E_Logo:Logo_8
- SW1: footprint EE:SW_PUSH_SMALL_2pin_3D_xl -> Explore:SW_PUSH_SMALL_2pin_3D_xl_v1
- U1: footprint EE:cp2102_xl2 -> Explore:cp2102_xl2
- X1: footprint Crystals:HC-49V -> Crystals:Crystal_HC18-U_Vertical
- moved P7 8.51 mm to (197.0, 117.2)
- moved CON1 1.52 mm to (196.8, 109.6)
- moved C3 0.38 mm to (190.4, 143.5)
- moved C2 0.25 mm to (203.2, 143.5)
Routing:
- net GND: track 180.4 -> 182.4 mm
- net /+5V: track 123.6 -> 125.1 mm
- net Net-(CON1-Pad3): track 4.64 -> 6.19 mm
- net Net-(CON1-Pad2): track 6.19 -> 7.74 mm
Other:
- outline, holes or cut-outs redrawn
- board text added: "oneMicro"
- board text removed: "PWR"

Commit message: Schematic PDF added
Routing:
- net /+5V: track 125.1 -> 129.3 mm
Changed lines of the file:
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@@
     (area 184.099999 104.724999 209.600001 167.690001)
     (thickness 1.6)
-    (drawings 84)
-    (tracks 628)
+    (drawings 80)
+    (tracks 629)
     (zones 0)
     (modules 30)
@@
   )
   (setup
-    (last_trace_width 0.254)
+    (last_trace_width 0.635)
     (user_trace_width 0.3048)
     (user_trace_width 0.381)
@@
     (add_net "Net-(IC1-Pad44)")
     (add_net "Net-(P1-Pad3)")
-    (add_net "Net-(P10-Pad1)")
-    (add_net "Net-(P6-Pad1)")
-    (add_net "Net-(P8-Pad1)")
-    (add_net "Net-(P9-Pad1)")
     (add_net "Net-(R4-Pad2)")
     (add_net "Net-(R5-Pad2)")
@@
     (tags "capacitor 0603")
     (attr smd)
-    (fp_text reference C2 (at 2.286 0 360) (layer F.SilkS)
+    (fp_text reference C2 (at -3.302 0 360) (layer F.SilkS)
       (effects (font (size 0.5842 0.5842) (thickness 0.14605)))
     )
@@
     (tags "capacitor 0603")
     (attr smd)
-    (fp_text reference C3 (at 2.286 0 360) (layer F.SilkS)
+    (fp_text reference C3 (at -3.302 0.127 360) (layer F.SilkS)
       (effects (font (size 0.5842 0.5842) (thickness 0.14605)))
     )
@@
     (tags "resistor 0603")
     (attr smd)
-    (fp_text reference R3 (at 0 -1.9 270) (layer F.SilkS) hide
-      (effects (font (size 1 1) (thickness 0.15)))
+    (fp_text reference R3 (at 2.4638 0.0762 360) (layer F.SilkS)
+      (effects (font (size 0.5842 0.5842) (thickness 0.14605)))
     )
     (fp_text value 470r (at 0 1.9 270) (layer F.Fab)
@@
     (tags "capacitor 0603")
     (attr smd)
-    (fp_text reference C8 (at 0 -1.9 270) (layer F.SilkS) hide
-      (effects (font (size 1 1) (thickness 0.15)))
+    (fp_text reference C8 (at 2.2606 0 360) (layer F.SilkS)
+      (effects (font (size 0.5842 0.5842) (thickness 0.14605)))
     )
     (fp_text value 0.1uF (at 0 1.9 270) (layer F.Fab)
@@
     (tags "capacitor 0603")
     (attr smd)
-    (fp_text reference C9 (at 2.159 0 180) (layer F.SilkS)
+    (fp_text reference C9 (at 2.794 0 180) (layer F.SilkS)
       (effects (font (size 0.5842 0.5842) (thickness 0.14605)))
     )
@@
     (effects (font (size 1.27 1.27) (thickness 0.3)) (justify mirror))
   )
-  (dimension 12.7 (width 0.3) (layer Eco2.User)
-    (gr_text "0.5000 in" (at 190.5 91.36) (layer Eco2.User)
-      (effects (font (size 1.5 1.5) (thickness 0.3)))
-    )
-    (feature1 (pts (xy 196.85 101.6) (xy 196.85 90.01)))
-    (feature2 (pts (xy 184.15 101.6) (xy 184.15 90.01)))
-    (crossbar (pts (xy 184.15 92.71) (xy 196.85 92.71)))
-    (arrow1a (pts (xy 196.85 92.71) (xy 195.723496 93.296421)))
-    (arrow1b (pts (xy 196.85 92.71) (xy 195.723496 92.123579)))
-    (arrow2a (pts (xy 184.15 92.71) (xy 185.276504 93.296421)))
-    (arrow2b (pts (xy 184.15 92.71) (xy 185.276504 92.123579)))
-  )
-  (dimension 25.4 (width 0.3) (layer Eco2.User)
-    (gr_text "1.0000 in" (at 196.85 97.71) (layer Eco2.User)
-      (effects (font (size 1.5 1.5) (thickness 0.3)))
-    )
-    (feature1 (pts (xy 209.55 102.87) (xy 209.55 96.36)))
-    (feature2 (pts (xy 184.15 102.87) (xy 184.15 96.36)))
-    (crossbar (pts (xy 184.15 99.06) (xy 209.55 99.06)))
-    (arrow1a (pts (xy 209.55 99.06) (xy 208.423496 99.646421)))
-    (arrow1b (pts (xy 209.55 99.06) (xy 208.423496 98.473579)))
-    (arrow2a (pts (xy 184.15 99.06) (xy 185.276504 99.646421)))
-    (arrow2b (pts (xy 184.15 99.06) (xy 185.276504 98.473579)))
-  )
   (gr_text SDA (at 205.486 138.43) (layer F.SilkS)
     (effects (font (size 1.016 1.016) (thickness 0.254)))
-  )
-  (dimension 22.86 (width 0.3) (layer Eco2.User)
-    (gr_text "0.9000 in" (at 196.85 79.93) (layer Eco2.User)
-      (effects (font (size 1.5 1.5) (thickness 0.3)))
-    )
-    (feature1 (pts (xy 208.28 93.98) (xy 208.28 78.58)))
-    (feature2 (pts (xy 185.42 93.98) (xy 185.42 78.58)))
-    (crossbar (pts (xy 185.42 81.28) (xy 208.28 81.28)))
-    (arrow1a (pts (xy 208.28 81.28) (xy 207.153496 81.866421)))
-    (arrow1b (pts (xy 208.28 81.28) (xy 207.153496 80.693579)))
-    (arrow2a (pts (xy 185.42 81.28) (xy 186.546504 81.866421)))
-    (arrow2b (pts (xy 185.42 81.28) (xy 186.546504 80.693579)))
-  )
-  (dimension 22.86 (width 0.3) (layer Eco2.User)
-    (gr_text "0.9000 in" (at 191.77 72.31) (layer Eco2.User)
-      (effects (font (size 1.5 1.5) (thickness 0.3)))
-    )
-    (feature1 (pts (xy 203.2 78.74) (xy 203.2 70.96)))
-    (feature2 (pts (xy 180.34 78.74) (xy 180.34 70.96)))
-    (crossbar (pts (xy 180.34 73.66) (xy 203.2 73.66)))
-    (arrow1a (pts (xy 203.2 73.66) (xy 202.073496 74.246421)))
-    (arrow1b (pts (xy 203.2 73.66) (xy 202.073496 73.073579)))
-    (arrow2a (pts (xy 180.34 73.66) (xy 181.466504 74.246421)))
-    (arrow2b (pts (xy 180.34 73.66) (xy 181.466504 73.073579)))
   )
   (gr_text Aref (at 187.96 135.89) (layer F.SilkS)
@@
     (effects (font (size 1.016 1.016) (thickness 0.254)))
   )
+  (segment (start 193.8274 157.7086) (end 199.4916 157.7086) (width 0.635) (layer B.Cu) (net 1))
+  (segment (start 200.449 157.564) (end 201.93 157.564) (width 0.635) (layer F.Cu) (net 1) (status 800000))
+  (segment (start 199.898 158.115) (end 200.449 157.564) (width 0.635) (layer F.Cu) (net 1))
+  (via (at 199.898 158.115) (size 0.91) (drill 0.5) (layers F.Cu B.Cu) (net 1))
+  (segment (start 199.4916 157.7086) (end 199.898 158.115) (width 0.635) (layer B.Cu) (net 1))
   (segment (start 198.15 111.252) (end 198.15 109.701) (width 0.381) (layer F.Cu) (net 1))
   (segment (start 198.308 123.444) (end 198.9328 123.444) (width 0.508) (layer F.Cu) (net 1))
@@
   (segment (start 195.5546 156.4132) (end 195.5546 154.5844) (width 0.635) (layer F.Cu) (net 1))
   (segment (start 194.2592 157.7086) (end 195.5546 156.4132) (width 0.635) (layer F.Cu) (net 1))
-  (segment (start 201.93 157.564) (end 198.4932 157.564) (width 0.635) (layer F.Cu) (net 1))
   (segment (start 193.5328 157.414) (end 191.77 157.414) (width 0.635) (layer F.Cu) (net 1))
   (segment (start 193.8274 157.7086) (end 193.5328 157.414) (width 0.635) (layer F.Cu) (net 1))
   (via (at 193.8274 157.7086) (size 0.91) (drill 0.5) (layers F.Cu B.Cu) (net 1))
   (segment (start 197.8406 157.7086) (end 193.8274 157.7086) (width 0.635) (layer B.Cu) (net 1))
-  (segment (start 198.0946 157.9626) (end 197.8406 157.7086) (width 0.635) (layer B.Cu) (net 1))
-  (via (at 198.0946 157.9626) (size 0.91) (drill 0.5) (layers F.Cu B.Cu) (net 1))
-  (segment (start 198.4932 157.564) (end 198.0946 157.9626) (width 0.635) (layer F.Cu) (net 1))
   (segment (start 201.93 165.735) (end 203.454 165.735) (width 0.635) (layer F.Cu) (net 1))
+  (segment (start 203.454 165.735) (end 204.1398 165.0492) (width 0.635) (layer F.Cu) (net 1))
+  (segment (start 204.1398 165.0492) (end 204.1398 161.29) (width 0.635) (layer F.Cu) (net 1))
+  (segment (start 204.1398 161.29) (end 201.93 159.0802) (width 0.635) (layer F.Cu) (net 1))
   (segment (start 201.93 159.0802) (end 201.93 157.564) (width 0.635) (layer F.Cu) (net 1))
-  (segment (start 204.1398 161.29) (end 201.93 159.0802) (width 0.635) (layer F.Cu) (net 1))
-  (segment (start 204.1398 165.0492) (end 204.1398 161.29) (width 0.635) (layer F.Cu) (net 1))
-  (segment (start 203.454 165.735) (end 204.1398 165.0492) (width 0.635) (layer F.Cu) (net 1))
   (segment (start 191 131.788) (end 189.4206 131.788) (width 0.381) (layer F.Cu) (net 1))
   (segment (start 189.0166 131.384) (end 188.468 131.384) (width 0.635) (layer F.Cu) (net 1))
@@
     (connect_pads (clearance 0.508))
     (min_thickness 0.254)
-    (fill yes (arc_segments 16) (thermal_gap 0.508) (thermal_bridge_width 0.508))
+    (fill (arc_segments 16) (thermal_gap 0.508) (thermal_bridge_width 0.508))
     (polygon
       (pts
@@
     (connect_pads (clearance 0.508))
     (min_thickness 0.254)
-    (fill yes (arc_segments 16) (thermal_gap 0.508) (thermal_bridge_width 0.508))
+    (fill (arc_segments 16) (thermal_gap 0.508) (thermal_bridge_width 0.508))
     (polygon
       (pts
