File: DesignFiles/40pin_AVRMCU.sch (KiCad schematic (older format))
At the start: 30 parts, among them CON1 USB-MINI-B, IC1 ATMEGA32-A, P1 CONN_5X2, P10 CONN_01X01, P2 CONN_10, P3 CONN_10, P4 CONN_10, P5 CONN_10, P6 CONN_01X01, P7 CONN_01X01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

Commit message: Changes done
Parts:
- C2, C3, C4, C5, C6, C7, C8, C9: footprint (none) -> Capacitors_SMD:C_0603_HandSoldering; symbol C -> C-RESCUE-40pin_AVRMCU
- CON1: footprint (none) -> Explore:USB_Micro-B_SMD_NEW_1
- D1, D3: footprint ~ -> Explore:LED-0603_NEW; symbol LED -> LED-RESCUE-40pin_AVRMCU
- IC1: footprint TQFP44 -> Housings_QFP:TQFP-44_10x10mm_Pitch0.8mm
- P1: footprint (none) -> Pin_Headers:Pin_Header_Straight_2x05_Pitch2.54mm
- P10, P6, P8, P9: footprint (none) -> Connect:1pin
- P2, P3, P4, P5: footprint (none) -> Pin_Headers:Pin_Header_Straight_1x10_Pitch2.54mm
- P7: footprint (none) -> E_Logo:Logo_8
- R1, R4, R5: footprint (none) -> Resistors_SMD:R_0603_HandSoldering; symbol R -> R-RESCUE-40pin_AVRMCU
- R2, R3: footprint ~ -> Resistors_SMD:R_0603_HandSoldering; symbol R -> R-RESCUE-40pin_AVRMCU
- SW1: footprint (none) -> Explore:SW_PUSH_SMALL_2pin_3D_xl_v1
- U1: footprint (none) -> Explore:cp2102_xl2
- X1: footprint (none) -> Crystals:Crystal_HC18-U_Vertical
Connections:
- net GND: now also D1.2 (K)
- net TX: now also D3.1 (A)
- net at R2.2: now also D1.1 (A)
- net at D3.2 (K): now also R3.1
Changed lines of the file:
@@
 EESchema Schematic File Version 2
+LIBS:40pin_AVRMCU-rescue
 LIBS:power
 LIBS:device
@@
 LIBS:memory
 LIBS:xilinx
-LIBS:special
 LIBS:microcontrollers
 LIBS:dsp
@@
 +5V
 $Comp
-L C C3
+L C-RESCUE-40pin_AVRMCU C3
 U 1 1 54F1C106
 P 2675 2350
 F 0 "C3" H 2725 2450 50  0000 L CNN
 F 1 "22pF" H 2725 2250 50  0000 L CNN
-F 2 "" H 2675 2350 60  0001 C CNN
+F 2 "Capacitors_SMD:C_0603_HandSoldering" H 2675 2350 60  0001 C CNN
 F 3 "" H 2675 2350 60  0001 C CNN
 	1    2675 2350
@@
 F 0 "P1" H 8625 1675 60  0000 C CNN
 F 1 "CONN_5X2" V 8625 1375 50  0000 C CNN
-F 2 "" H 8625 1375 60  0001 C CNN
+F 2 "Pin_Headers:Pin_Header_Straight_2x05_Pitch2.54mm" H 8625 1375 60  0001 C CNN
 F 3 "" H 8625 1375 60  0001 C CNN
 	1    8625 1375
@@
 F 0 "SW1" H 1675 3975 70  0000 C CNN
 F 1 "rst" H 1675 3775 70  0000 C CNN
-F 2 "" H 1675 3875 60  0001 C CNN
+F 2 "Explore:SW_PUSH_SMALL_2pin_3D_xl_v1" H 1675 3875 60  0001 C CNN
 F 3 "" H 1675 3875 60  0001 C CNN
 	1    1675 3875
@@
 $EndComp
 $Comp
-L C C4
+L C-RESCUE-40pin_AVRMCU C4
 U 1 1 54F1C148
 P 3025 2900
 F 0 "C4" H 3075 3000 50  0000 L CNN
 F 1 "0.1uF" H 3075 2800 50  0000 L CNN
-F 2 "" H 3025 2900 60  0001 C CNN
+F 2 "Capacitors_SMD:C_0603_HandSoldering" H 3025 2900 60  0001 C CNN
 F 3 "" H 3025 2900 60  0001 C CNN
 	1    3025 2900
@@
 $EndComp
 $Comp
-L C C6
+L C-RESCUE-40pin_AVRMCU C6
 U 1 1 54F1C154
 P 4525 950
 F 0 "C6" H 4575 1050 50  0000 L CNN
 F 1 "0.1uF" H 4425 850 50  0000 L CNN
-F 2 "" H 4525 950 60  0001 C CNN
+F 2 "Capacitors_SMD:C_0603_HandSoldering" H 4525 950 60  0001 C CNN
 F 3 "" H 4525 950 60  0001 C CNN
 	1    4525 950
@@
 $EndComp
 $Comp
-L C C2
+L C-RESCUE-40pin_AVRMCU C2
 U 1 1 54F1C167
 P 2675 1750
 F 0 "C2" H 2725 1850 50  0000 L CNN
 F 1 "22pF" H 2725 1650 50  0000 L CNN
-F 2 "" H 2675 1750 60  0001 C CNN
+F 2 "Capacitors_SMD:C_0603_HandSoldering" H 2675 1750 60  0001 C CNN
 F 3 "" H 2675 1750 60  0001 C CNN
 	1    2675 1750
@@
 F 0 "X1" H 2925 2200 60  0000 C CNN
 F 1 "16Mhz" H 2925 1900 60  0000 C CNN
-F 2 "" H 2925 2050 60  0001 C CNN
+F 2 "Crystals:Crystal_HC18-U_Vertical" H 2925 2050 60  0001 C CNN
 F 3 "" H 2925 2050 60  0001 C CNN
 	1    2925 2050
@@
 rst
 $Comp
-L R R1
+L R-RESCUE-40pin_AVRMCU R1
 U 1 1 54F1C18C
 P 1675 3025
 F 0 "R1" V 1755 3025 50  0000 C CNN
 F 1 "10K" V 1675 3025 50  0000 C CNN
-F 2 "" H 1675 3025 60  0001 C CNN
+F 2 "Resistors_SMD:R_0603_HandSoldering" H 1675 3025 60  0001 C CNN
 F 3 "" H 1675 3025 60  0001 C CNN
 	1    1675 3025
@@
 $EndComp
 $Comp
-L C C5
+L C-RESCUE-40pin_AVRMCU C5
 U 1 1 54F1C1A0
 P 4525 650
 F 0 "C5" H 4575 750 50  0000 L CNN
 F 1 "0.1uF" H 4575 550 50  0000 L CNN
-F 2 "" H 4525 650 60  0001 C CNN
+F 2 "Capacitors_SMD:C_0603_HandSoldering" H 4525 650 60  0001 C CNN
 F 3 "" H 4525 650 60  0001 C CNN
 	1    4525 650
@@
 F 0 "P5" V 6525 2600 60  0000 C CNN
 F 1 "CONN_10" V 6625 2600 60  0000 C CNN
-F 2 "" H 6575 2600 60  0000 C CNN
+F 2 "Pin_Headers:Pin_Header_Straight_1x10_Pitch2.54mm" H 6575 2600 60  0001 C CNN
 F 3 "" H 6575 2600 60  0000 C CNN
 	1    6575 2600
@@
 F 0 "P3" V 6525 1500 60  0000 C CNN
 F 1 "CONN_10" V 6625 1500 60  0000 C CNN
-F 2 "" H 6575 1500 60  0000 C CNN
+F 2 "Pin_Headers:Pin_Header_Straight_1x10_Pitch2.54mm" H 6575 1500 60  0001 C CNN
 F 3 "" H 6575 1500 60  0000 C CNN
 	1    6575 1500
@@
 F 0 "P2" V 6125 4500 60  0000 C CNN
 F 1 "CONN_10" V 6225 4500 60  0000 C CNN
-F 2 "" H 6175 4500 60  0000 C CNN
+F 2 "Pin_Headers:Pin_Header_Straight_1x10_Pitch2.54mm" H 6175 4500 60  0001 C CNN
 F 3 "" H 6175 4500 60  0000 C CNN
 	1    6175 4500
@@
 F 0 "P4" V 7225 3700 60  0000 C CNN
 F 1 "CONN_10" V 7325 3700 60  0000 C CNN
-F 2 "" H 7275 3700 60  0000 C CNN
+F 2 "Pin_Headers:Pin_Header_Straight_1x10_Pitch2.54mm" H 7275 3700 60  0001 C CNN
 F 3 "" H 7275 3700 60  0000 C CNN
 	1    7275 3700
@@
 $EndComp
 $Comp
-L R R2
+L R-RESCUE-40pin_AVRMCU R2
 U 1 1 54F94C0B
 P 1675 1075
 F 0 "R2" V 1755 1075 40  0000 C CNN
 F 1 "470r" V 1682 1076 40  0000 C CNN
-F 2 "~" V 1605 1075 30  0000 C CNN
+F 2 "Resistors_SMD:R_0603_HandSoldering" V 1605 1075 30  0000 C CNN
 F 3 "~" H 1675 1075 30  0000 C CNN
 	1    1675 1075
@@
 $EndComp
 $Comp
-L LED D1
+L LED-RESCUE-40pin_AVRMCU D1
 U 1 1 54F94C1A
 P 1675 1625
 F 0 "D1" H 1675 1725 50  0000 C CNN
 F 1 "LED" H 1675 1525 50  0000 C CNN
-F 2 "~" H 1675 1625 60  0000 C CNN
+F 2 "Explore:LED-0603_NEW" H 1675 1625 60  0000 C CNN
 F 3 "~" H 1675 1625 60  0000 C CNN
 	1    1675 1625
@@
 +5V
 $Comp
-L LED D3
+L LED-RESCUE-40pin_AVRMCU D3
 U 1 1 5514EDCE
 P 8275 2300
 F 0 "D3" H 8275 2400 50  0000 C CNN
 F 1 "LED" H 8275 2200 50  0000 C CNN
-F 2 "~" H 8275 2300 60  0000 C CNN
+F 2 "Explore:LED-0603_NEW" H 8275 2300 60  0000 C CNN
 F 3 "~" H 8275 2300 60  0000 C CNN
 	1    8275 2300
@@
 $EndComp
 $Comp
-L R R3
+L R-RESCUE-40pin_AVRMCU R3
 U 1 1 5514EDD4
 P 8825 2300
 F 0 "R3" V 8905 2300 40  0000 C CNN
 F 1 "470r" V 8832 2301 40  0000 C CNN
-F 2 "~" V 8755 2300 30  0000 C CNN
+F 2 "Resistors_SMD:R_0603_HandSoldering" V 8755 2300 30  0000 C CNN
 F 3 "~" H 8825 2300 30  0000 C CNN
 	1    8825 2300
@@
 F 0 "IC1" H 3325 5030 40  0000 L BNN
 F 1 "ATMEGA32-A" H 4625 1200 40  0000 L BNN
-F 2 "TQFP44" H 4175 3150 30  0000 C CIN
+F 2 "Housings_QFP:TQFP-44_10x10mm_Pitch0.8mm" H 4175 3150 30  0000 C CIN
 F 3 "" H 4175 3150 60  0000 C CNN
 	1    4175 3150
@@
 F 0 "P7" H 9125 4550 50  0000 C CNN
 F 1 "CONN_01X01" V 9225 4450 50  0000 C CNN
-F 2 "" H 9125 4450 60  0000 C CNN
+F 2 "E_Logo:Logo_8" H 9125 4450 60  0001 C CNN
 F 3 "" H 9125 4450 60  0000 C CNN
 	1    9125 4450
@@
 F 0 "CON1" H 1550 6900 50  0000 C CNN
 F 1 "USB-MINI-B" H 1700 6200 50  0000 C CNN
-F 2 "" H 1850 6450 50  0000 C CNN
+F 2 "Explore:USB_Micro-B_SMD_NEW_1" H 1850 6450 50  0001 C CNN
 F 3 "" H 1850 6450 50  0000 C CNN
 	1    1850 6550
@@
 	2350 6550 2950 6550
 $Comp
-L C C8
+L C-RESCUE-40pin_AVRMCU C8
 U 1 1 579B2BB0
 P 3050 7300
 F 0 "C8" H 3100 7400 50  0000 L CNN
 F 1 "0.1uF" H 3100 7200 50  0000 L CNN
-F 2 "" H 3050 7300 60  0001 C CNN
+F 2 "Capacitors_SMD:C_0603_HandSoldering" H 3050 7300 60  0001 C CNN
 F 3 "" H 3050 7300 60  0001 C CNN
 	1    3050 7300
@@
 	2950 6350 2950 5500
 $Comp
-L C C7
+L C-RESCUE-40pin_AVRMCU C7
 U 1 1 579B3250
 P 2650 5800
 F 0 "C7" H 2700 5900 50  0000 L CNN
 F 1 "0.1uF" H 2700 5700 50  0000 L CNN
-F 2 "" H 2650 5800 60  0001 C CNN
+F 2 "Capacitors_SMD:C_0603_HandSoldering" H 2650 5800 60  0001 C CNN
 F 3 "" H 2650 5800 60  0001 C CNN
 	1    2650 5800
@@
 F 0 "U1" H 3650 6500 60  0000 C CNN
 F 1 "CP2102" H 4300 6500 60  0000 C CNN
-F 2 "" H 3650 6500 60  0000 C CNN
+F 2 "Explore:cp2102_xl2" H 3650 6500 60  0001 C CNN
 F 3 "" H 3650 6500 60  0000 C CNN
 	1    4200 6500
@@
 $EndComp
 $Comp
-L R R5
+L R-RESCUE-40pin_AVRMCU R5
 U 1 1 579B3A3A
 P 5950 6450
 F 0 "R5" V 6030 6450 50  0000 C CNN
 F 1 "470" V 5957 6451 50  0000 C CNN
-F 2 "" V 5880 6450 30  0000 C CNN
+F 2 "Resistors_SMD:R_0603_HandSoldering" V 5880 6450 30  0001 C CNN
 F 3 "" H 5950 6450 30  0000 C CNN
 	1    5950 6450
@@
 RX
 $Comp
-L C C9
+L C-RESCUE-40pin_AVRMCU C9
 U 1 1 579B4297
 P 6400 6550
 F 0 "C9" H 6450 6650 50  0000 L CNN
 F 1 "0.1uF" H 6450 6450 50  0000 L CNN
-F 2 "" H 6400 6550 60  0001 C CNN
+F 2 "Capacitors_SMD:C_0603_HandSoldering" H 6400 6550 60  0001 C CNN
 F 3 "" H 6400 6550 60  0001 C CNN
 	1    6400 6550
@@
 F 0 "P6" H 9925 4525 50  0000 C CNN
 F 1 "CONN_01X01" V 10025 4425 50  0000 C CNN
-F 2 "" H 9925 4425 60  0000 C CNN
+F 2 "Connect:1pin" H 9925 4425 60  0001 C CNN
 F 3 "" H 9925 4425 60  0000 C CNN
 	1    9925 4425
@@
 F 0 "P9" H 10600 4525 50  0000 C CNN
 F 1 "CONN_01X01" V 10700 4425 50  0000 C CNN
-F 2 "" H 10600 4425 60  0000 C CNN
+F 2 "Connect:1pin" H 10600 4425 60  0001 C CNN
 F 3 "" H 10600 4425 60  0000 C CNN
 	1    10600 4425
@@
 F 0 "P8" H 9925 5200 50  0000 C CNN
 F 1 "CONN_01X01" V 10025 5100 50  0000 C CNN
-F 2 "" H 9925 5100 60  0000 C CNN
+F 2 "Connect:1pin" H 9925 5100 60  0001 C CNN
 F 3 "" H 9925 5100 60  0000 C CNN
 	1    9925 5100
@@
 F 0 "P10" H 10600 5200 50  0000 C CNN
 F 1 "CONN_01X01" V 10700 5100 50  0000 C CNN
-F 2 "" H 10600 5100 60  0000 C CNN
+F 2 "Connect:1pin" H 10600 5100 60  0001 C CNN
 F 3 "" H 10600 5100 60  0000 C CNN
 	1    10600 5100
@@
 NoConn ~ 2350 6650
 $Comp
-L R R4
+L R-RESCUE-40pin_AVRMCU R4
 U 1 1 579C4A4D
 P 5700 6350
 F 0 "R4" V 5780 6350 50  0000 C CNN
 F 1 "470" V 5707 6351 50  0000 C CNN
-F 2 "" V 5630 6350 30  0000 C CNN
+F 2 "Resistors_SMD:R_0603_HandSoldering" V 5630 6350 30  0001 C CNN
 F 3 "" H 5700 6350 30  0000 C CNN
 	1    5700 6350

Commit message: Schematic PDF added
Parts:
- D1, D3: footprint Explore:LED-0603_NEW -> LED; symbol LED-RESCUE-40pin_AVRMCU -> LED
- R2, R3: footprint Resistors_SMD:R_0603_HandSoldering -> Resistors
Connections:
- net TX: no longer D3.1 (A)
- net at D3.2 (A): no longer R3.1
Other:
- note added: "Controller"
- note added: "USB to Serial"
- note removed: "Breakout for USB to Serial"
- moved on the sheet: C2, C3, C4, C5, C6, C7, C8, C9, CON1, D1, D3, IC1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
